File: Prototype/Eagle/Motherboard/AmbaSat-1v1-01-NO-solar.brd (EAGLE design)
At the start: 37 x 35 mm, 18 parts, among them J1 SCK MISO MOSI D3 SDA SCL GND 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, U1 LSM9DS1

Commit message: C1 modification
Value of C1 not displayed. Also incorrect. Was 1uF. Should be 0.1uF
Parts:
- C1: value 1uF -> 0.1uF
Changed lines of the file:
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@@
 <attribute name="VALUE" x="13.635" y="23.5456" size="0.6096" layer="27" ratio="6" rot="SR90"/>
 </element>
-<element name="C1" library="rcl" package="C0805K" value="1uF" x="2" y="17.7" smashed="yes" rot="R270">
+<element name="C1" library="rcl" package="C0805K" value="0.1uF" x="2" y="17.7" smashed="yes" rot="R270">
 <attribute name="NAME" x="1.4" y="19.675" size="0.8128" layer="25" font="vector" ratio="18"/>
 <attribute name="VALUE" x="0.1" y="18.7" size="1.016" layer="27" rot="R270"/>
