File: Prototype/Eagle/Motherboard/AmbaSat-1v1-01-NO-solar.sch (EAGLE design)
At the start: 18 parts, among them J1 SCK MISO MOSI D3 SDA SCL GND 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, U1 LSM9DS1

Commit message: C1 modification
Value of C1 not displayed. Also incorrect. Was 1uF. Should be 0.1uF
Parts:
- C1: value 1uF -> 0.1uF
Changed lines of the file:
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@@
 <part name="R1" library="rcl" deviceset="R-EU_" device="M0805" value=" 1k6"/>
 <part name="R2" library="rcl" deviceset="R-EU_" device="M0805" value=" 10k"/>
-<part name="C1" library="rcl" deviceset="C-EU" device="C0805K" value="1uF"/>
+<part name="C1" library="rcl" deviceset="C-EU" device="C0805K" value="0.1uF"/>
 <part name="GND2" library="supply1" deviceset="GND" device=""/>
 <part name="GND3" library="supply1" deviceset="GND" device=""/>
@@
 <instance part="R2" gate="G$1" x="78.74" y="160.02"/>
 <instance part="C1" gate="G$1" x="68.58" y="91.44" smashed="yes" rot="R270">
-<attribute name="NAME" x="68.961" y="94.996" size="1.778" layer="95" font="vector"/>
+<attribute name="NAME" x="71.501" y="89.916" size="1.778" layer="95" rot="R180"/>
+<attribute name="VALUE" x="65.024" y="94.361" size="1.778" layer="96"/>
 </instance>
 <instance part="GND2" gate="1" x="17.78" y="119.38"/>
