File: Release/Eagle/Solarboard/SolarBoard version 2.01.sch (EAGLE design)
At the start: 6 parts

Commit message: Label updates - Schematic
Other:
- note added: "© 2020 AmbaSat Ltd Authors: John Mowbray, Martin Platt, Sudu Malli Web: ambasat.com"
- note removed: "AmbaSat-1 Solarboard"
