File: Release/Eagle/Motherboard/AmbaSat-1 version 2.02.sch (EAGLE design)
At the start: 22 parts, among them U1 LSM9DS1, Y1 4MHz

Commit message: Update AmbaSat-1 version 2.02.sch
Other:
- note added: "© 2020 AmbaSat Ltd Authors: John Mowbray, Martin Platt, Sudu Malli Web: ambasat.com"
- note removed: "© 2019 AmbaSat Ltd Authors: John M & Martin P"
Changed lines of the file:
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@@
 <?xml version="1.0" encoding="utf-8"?>
 <!DOCTYPE eagle SYSTEM "eagle.dtd">
-<eagle version="9.3.2">
+<eagle version="9.5.1">
 <drawing>
 <settings>
@@
 <text x="-22.86" y="33.02" size="3.81" layer="94" ratio="10">AmbaSat-1
 Sprite class satellite (ChipSat/Femtosatellite)</text>
-<text x="132.08" y="33.02" size="3.048" layer="94" ratio="10">© 2019 AmbaSat Ltd
-Authors: John M &amp; Martin P</text>
+<text x="132.08" y="33.02" size="2.54" layer="94" ratio="10">© 2020 AmbaSat Ltd
+Authors: John Mowbray,
+Martin Platt, Sudu Malli
+Web: ambasat.com</text>
 </plain>
 <instances>
