File: Release/KiCad/Motherboard/AmbaSat-1 Satellite.kicad_pcb (KiCad board)
At the start: 2 copper layers, 35 x 35 mm, 23 parts, among them U1 LSM9DS1, U2 ATMEGA328P-AU, U3 LP2985AIM5-3.3, U4 RFM95, Y1 4MHz

Commit message: Moves referenced symbols to separate library
The Eagle import included a number of symbols that were not used.
This commit moves only the referenced symbols to their own library, and
replaces some of the more generic Eagle symbols with their generic KiCad
counterparts (i.e. R, C, LED, 3V3, GND).
Connections:
- net VCC renamed 3V3
