File: Release/KiCad/Motherboard/AmbaSat-1 Satellite.sch (KiCad schematic (older format))
At the start: 22 parts, among them U1 LSM9DS1, U2 ATMEGA328P-AU, U3 LP2985AIM5-3.3, U4 RFM95, Y1 4MHz

Commit message: Moves referenced symbols to separate library
The Eagle import included a number of symbols that were not used.
This commit moves only the referenced symbols to their own library, and
replaces some of the more generic Eagle symbols with their generic KiCad
counterparts (i.e. R, C, LED, 3V3, GND).
Parts:
- C1, C3, C4, C5, C6, C7, C8, C9: symbol AmbaSat-1_Satellite-eagle-import:C-EUC0805K -> AmbaSat-1_Satellite-Symbols:C
- D1: symbol AmbaSat-1_Satellite-eagle-import:LEDCHIP-LED0805 -> AmbaSat-1_Satellite-Symbols:LED
- JP1: symbol AmbaSat-1_Satellite-eagle-import:PINHD-1X8 -> AmbaSat-1_Satellite-Symbols:PINHD-1X8
- JP2: symbol AmbaSat-1_Satellite-eagle-import:PINHD-1X6 -> AmbaSat-1_Satellite-Symbols:PINHD-1X6
- JP3: symbol AmbaSat-1_Satellite-eagle-import:HEADER-1X1ROUND -> AmbaSat-1_Satellite-Symbols:HEADER-1X1ROUND
- R1, R2, R3, R4: symbol AmbaSat-1_Satellite-eagle-import:R-EU_M0805 -> AmbaSat-1_Satellite-Symbols:R
- U.FL1: symbol AmbaSat-1_Satellite-eagle-import:U.FL -> AmbaSat-1_Satellite-Symbols:U.FL
- U1: symbol AmbaSat-1_Satellite-eagle-import:LSM9DS1 -> AmbaSat-1_Satellite-Symbols:LSM9DS1
- U2: symbol AmbaSat-1_Satellite-eagle-import:ATMEGA328P-AU -> AmbaSat-1_Satellite-Symbols:ATMEGA328P-AU
- U3: symbol AmbaSat-1_Satellite-eagle-import:LP2985AIM5-3.3 -> AmbaSat-1_Satellite-Symbols:LP2985AIM5-3.3
- U4: symbol AmbaSat-1_Satellite-eagle-import:RFM95 -> AmbaSat-1_Satellite-Symbols:RFM95
- Y1: symbol AmbaSat-1_Satellite-eagle-import:RESONATOR-4MHZSMD-4.5X2 -> AmbaSat-1_Satellite-Symbols:RESONATOR-4MHZSMD-4.5X2
Connections:
- net labels added: 3V3
- net labels removed: VCC
- wire segments 131 -> 134
